File: schematic/base.sch (EAGLE design)
At the start: 7 parts, among them IC1 MEGA328-PU

Commit message: Add files via upload
Parts:
- added C2: 100n, rcl:C-EU025-025X050
- added JP5: GY-NEO6MV2, pinhead:PINHD-1X4
- added LDR1: GL5528, photo-elements:VT20N1
- added R2: 10K, rcl:R-EU_0204/7
Connections:
- new net N$13: IC1.PC2(ADC2/PCINT10), LDR1.1, R2.1
- new net N$14: IC1.PB0(ICP1/CLKO/PCINT0), JP5.2
- new net N$15: IC1.PB1(OC1A/PCINT1), JP5.3
- new net N$4: C2.1, IC1.AREF
- net +3V3: now also IC1.AVCC, JP5.1, R2.2
- net GND: now also C2.2, IC1.AGND, JP5.4, LDR1.2
- net N$10: now also IC1.PD4(T0/XCK/PCINT20); no longer IC1.PD7(AIN1/PCINT23)
- net N$6: now also IC1.PD6(AIN0/OC0A/PCINT22); no longer IC1.PB0(ICP1/CLKO/PCINT0)
- net N$7: now also IC1.PD7(AIN1/PCINT23); no longer IC1.PB1(OC1A/PCINT1)
Other:
- note added: "VCC RX TX GND"
- moved on the sheet: C1, JP2, JP3, JP4, R1

Commit message: Add files via upload
Parts:
- added JP6: RS232, pinhead:PINHD-1X3
- added R3, R4: 10K, rcl:R-EU_0204/7
- JP3: device pinhead:PINHD-1X9 -> pinhead:PINHD-1X14
Connections:
- new net N$16: IC1.PD3(INT1/OC2B/PCINT19), JP3.11, R3.1
- new net N$17: IC1.PD1(TXD/PCINT17), JP6.2
- net +3V3: now also R1.2, R3.2, R4.2; no longer R1.1
- net GND: now also JP6.1
- net N$1: now also IC1.PB2(SS/OC1B/PCINT2), JP2.5; no longer IC1.PC4(ADC4/SDA/PCINT12), JP2.4
- net N$12: now also JP2.3, JP3.10
- net N$2: now also R1.1; no longer R1.2
- net N$3: now also IC1.PB4(MISO/PCINT4), JP1.9, JP2.6, JP3.13, JP3.9; no longer IC1.PC5(ADC5/SCLPCINT13), JP2.3
- net N$7: now also R4.1
- net N$8: now also JP2.4, JP3.12
- net N$9: now also IC1.PD2(INT0/PCINT18), JP3.14; no longer IC1.PB4(MISO/PCINT4), JP1.9, JP3.9
Other:
- note added: "GND TXD RXD"
- note added: "VCC GND CS RESET DC/RS SDI/MOSI SCK LED SDO/MISO T_CLK T_CS T_DIN T_DO T_IRQ"
- note removed: "VCC GND CS RESET DC/RS SDI/MOSI SCK LED SDO/MISO"
- moved on the sheet: JP2, JP4, JP5, LDR1, R1, R2

Commit message: Add files via upload
Parts:
- added C3, C4: 22p, rcl:C-EU025-025X050
- added Q1: 12MHz, crystal:CRYSTALHC49U-V
Connections:
- new net N$18: C4.1, IC1.PB7(XTAL2/TOSC2/PCINT7), Q1.1
- new net N$19: C3.1, IC1.PB6(XTAL1/TOSC1/PCINT6), Q1.2
- net GND: now also C3.2, C4.2
Other:
- moved on the sheet: C1
Changed lines of the file:
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@@
 <part name="R4" library="rcl" deviceset="R-EU_" device="0204/7" value="10K"/>
 <part name="JP6" library="pinhead" deviceset="PINHD-1X3" device="" value="RS232"/>
+<part name="Q1" library="crystal" deviceset="CRYSTAL" device="HC49U-V" value="12MHz"/>
+<part name="C3" library="rcl" deviceset="C-EU" device="025-025X050" value="22p"/>
+<part name="C4" library="rcl" deviceset="C-EU" device="025-025X050" value="22p"/>
 </parts>
 <sheets>
@@
 <instance part="JP1" gate="G$1" x="48.26" y="12.7"/>
 <instance part="IC1" gate="1" x="30.48" y="63.5"/>
-<instance part="+3V1" gate="G$1" x="-17.78" y="121.92"/>
-<instance part="GND1" gate="1" x="-17.78" y="-5.08"/>
-<instance part="C1" gate="G$1" x="-17.78" y="48.26"/>
+<instance part="+3V1" gate="G$1" x="-27.94" y="121.92"/>
+<instance part="GND1" gate="1" x="-27.94" y="-5.08"/>
+<instance part="C1" gate="G$1" x="-27.94" y="48.26"/>
 <instance part="R1" gate="G$1" x="-7.62" y="101.6" rot="R90"/>
 <instance part="JP2" gate="A" x="121.92" y="109.22"/>
@@
 <instance part="R4" gate="G$1" x="88.9" y="101.6" rot="R90"/>
 <instance part="JP6" gate="A" x="121.92" y="88.9"/>
+<instance part="Q1" gate="G$1" x="-2.54" y="73.66" rot="R90"/>
+<instance part="C3" gate="G$1" x="-20.32" y="48.26"/>
+<instance part="C4" gate="G$1" x="-12.7" y="48.26"/>
 </instances>
 <busses>
@@
 <segment>
 <pinref part="+3V1" gate="G$1" pin="+3V3"/>
-<wire x1="-17.78" y1="116.84" x2="-17.78" y2="119.38" width="0.1524" layer="91"/>
-<wire x1="-17.78" y1="116.84" x2="-7.62" y2="116.84" width="0.1524" layer="91"/>
+<wire x1="-27.94" y1="116.84" x2="-27.94" y2="119.38" width="0.1524" layer="91"/>
+<wire x1="-27.94" y1="116.84" x2="-7.62" y2="116.84" width="0.1524" layer="91"/>
 <wire x1="-7.62" y1="116.84" x2="66.04" y2="116.84" width="0.1524" layer="91"/>
 <wire x1="66.04" y1="116.84" x2="73.66" y2="116.84" width="0.1524" layer="91"/>
@@
 <junction x="88.9" y="116.84"/>
 <pinref part="IC1" gate="1" pin="VCC@1"/>
-<wire x1="0" y1="63.5" x2="-17.78" y2="63.5" width="0.1524" layer="91"/>
-<wire x1="-17.78" y1="55.88" x2="-17.78" y2="63.5" width="0.1524" layer="91"/>
+<wire x1="0" y1="63.5" x2="-27.94" y2="63.5" width="0.1524" layer="91"/>
+<wire x1="-27.94" y1="55.88" x2="-27.94" y2="63.5" width="0.1524" layer="91"/>
 <pinref part="IC1" gate="1" pin="AVCC"/>
-<wire x1="0" y1="55.88" x2="-17.78" y2="55.88" width="0.1524" layer="91"/>
-<junction x="-17.78" y="55.88"/>
+<wire x1="0" y1="55.88" x2="-27.94" y2="55.88" width="0.1524" layer="91"/>
+<junction x="-27.94" y="55.88"/>
 <pinref part="C1" gate="G$1" pin="1"/>
-<wire x1="-17.78" y1="50.8" x2="-17.78" y2="55.88" width="0.1524" layer="91"/>
-<wire x1="-17.78" y1="116.84" x2="-17.78" y2="63.5" width="0.1524" layer="91"/>
+<wire x1="-27.94" y1="50.8" x2="-27.94" y2="55.88" width="0.1524" layer="91"/>
+<wire x1="-27.94" y1="116.84" x2="-27.94" y2="63.5" width="0.1524" layer="91"/>
 <pinref part="R1" gate="G$1" pin="2"/>
 <wire x1="-7.62" y1="106.68" x2="-7.62" y2="116.84" width="0.1524" layer="91"/>
-<junction x="-17.78" y="63.5"/>
+<junction x="-27.94" y="63.5"/>
 <junction x="-7.62" y="116.84"/>
-<junction x="-17.78" y="116.84"/>
+<junction x="-27.94" y="116.84"/>
 </segment>
 </net>
@@
 <pinref part="IC1" gate="1" pin="GND@1"/>
 <pinref part="C1" gate="G$1" pin="2"/>
-<wire x1="0" y1="35.56" x2="-17.78" y2="35.56" width="0.1524" layer="91"/>
-<wire x1="-17.78" y1="35.56" x2="-17.78" y2="40.64" width="0.1524" layer="91"/>
+<wire x1="0" y1="35.56" x2="-12.7" y2="35.56" width="0.1524" layer="91"/>
+<wire x1="-12.7" y1="35.56" x2="-20.32" y2="35.56" width="0.1524" layer="91"/>
+<wire x1="-20.32" y1="35.56" x2="-27.94" y2="35.56" width="0.1524" layer="91"/>
+<wire x1="-27.94" y1="35.56" x2="-27.94" y2="40.64" width="0.1524" layer="91"/>
 <pinref part="GND1" gate="1" pin="GND"/>
-<wire x1="-17.78" y1="40.64" x2="-17.78" y2="43.18" width="0.1524" layer="91"/>
-<wire x1="-17.78" y1="-2.54" x2="-17.78" y2="0" width="0.1524" layer="91"/>
-<junction x="-17.78" y="35.56"/>
-<junction x="-17.78" y="0"/>
-<wire x1="-17.78" y1="0" x2="-17.78" y2="35.56" width="0.1524" layer="91"/>
+<wire x1="-27.94" y1="40.64" x2="-27.94" y2="43.18" width="0.1524" layer="91"/>
+<wire x1="-27.94" y1="-2.54" x2="-27.94" y2="0" width="0.1524" layer="91"/>
+<junction x="-27.94" y="35.56"/>
+<junction x="-27.94" y="0"/>
+<wire x1="-27.94" y1="0" x2="-27.94" y2="35.56" width="0.1524" layer="91"/>
 <pinref part="JP2" gate="A" pin="2"/>
 <wire x1="119.38" y1="114.3" x2="93.98" y2="114.3" width="0.1524" layer="91"/>
@@
 <junction x="93.98" y="66.04"/>
 <pinref part="JP1" gate="G$1" pin="3"/>
-<wire x1="40.64" y1="0" x2="-17.78" y2="0" width="0.1524" layer="91"/>
+<wire x1="40.64" y1="0" x2="-27.94" y2="0" width="0.1524" layer="91"/>
 <wire x1="43.18" y1="17.78" x2="40.64" y2="17.78" width="0.1524" layer="91"/>
 <wire x1="40.64" y1="17.78" x2="40.64" y2="15.24" width="0.1524" layer="91"/>
@@
 <pinref part="IC1" gate="1" pin="AGND"/>
 <wire x1="0" y1="40.64" x2="-2.54" y2="40.64" width="0.1524" layer="91"/>
-<junction x="-17.78" y="40.64"/>
+<junction x="-27.94" y="40.64"/>
 <pinref part="C2" gate="G$1" pin="2"/>
-<wire x1="-2.54" y1="40.64" x2="-17.78" y2="40.64" width="0.1524" layer="91"/>
+<wire x1="-2.54" y1="40.64" x2="-27.94" y2="40.64" width="0.1524" layer="91"/>
 <wire x1="-2.54" y1="43.18" x2="-2.54" y2="40.64" width="0.1524" layer="91"/>
 <junction x="-2.54" y="40.64"/>
@@
 <wire x1="119.38" y1="91.44" x2="93.98" y2="91.44" width="0.1524" layer="91"/>
 <junction x="93.98" y="91.44"/>
+<pinref part="C3" gate="G$1" pin="2"/>
+<wire x1="-20.32" y1="43.18" x2="-20.32" y2="35.56" width="0.1524" layer="91"/>
+<pinref part="C4" gate="G$1" pin="2"/>
+<wire x1="-12.7" y1="43.18" x2="-12.7" y2="35.56" width="0.1524" layer="91"/>
+<junction x="-20.32" y="35.56"/>
+<junction x="-12.7" y="35.56"/>
 </segment>
 </net>
@@
 </segment>
 </net>
+<net name="N$18" class="0">
+<segment>
+<pinref part="IC1" gate="1" pin="PB7(XTAL2/TOSC2/PCINT7)"/>
+<pinref part="C4" gate="G$1" pin="1"/>
+<wire x1="0" y1="71.12" x2="-2.54" y2="71.12" width="0.1524" layer="91"/>
+<wire x1="-2.54" y1="71.12" x2="-12.7" y2="71.12" width="0.1524" layer="91"/>
+<wire x1="-12.7" y1="71.12" x2="-12.7" y2="50.8" width="0.1524" layer="91"/>
+<pinref part="Q1" gate="G$1" pin="1"/>
+<junction x="-2.54" y="71.12"/>
+</segment>
+</net>
+<net name="N$19" class="0">
+<segment>
+<pinref part="IC1" gate="1" pin="PB6(XTAL1/TOSC1/PCINT6)"/>
+<pinref part="C3" gate="G$1" pin="1"/>
+<wire x1="0" y1="76.2" x2="-2.54" y2="76.2" width="0.1524" layer="91"/>
+<wire x1="-2.54" y1="76.2" x2="-20.32" y2="76.2" width="0.1524" layer="91"/>
+<wire x1="-20.32" y1="76.2" x2="-20.32" y2="50.8" width="0.1524" layer="91"/>
+<pinref part="Q1" gate="G$1" pin="2"/>
+<junction x="-2.54" y="76.2"/>
+</segment>
+</net>
