File: schematic/remote_25_45_85-1wire.sch (EAGLE design)
At the start: 8 parts, among them IC1 TINY25/45/85, IC2 DS18B20

Commit message: Add files via upload
Parts:
- added R3: 2K2, resistor:R-EU_0204/7
- added R4, R7: 4K7, resistor:R-EU_0204/7
- added R5: 10K, resistor:R-EU_0204/7
- added R6: 330, resistor:R-EU_0204/7
- R1: value 330 -> 560
- R2: value 4K7 -> 1K2
- S1: value Address -> (none); device switch-omron:10-XX -> switch-dil:DIP04S
Connections:
- new net N$10: R3.1, R4.2, S1-3.1, S1-4.1
- new net N$14: IC2_1W.1W, R6.1, R7.1
- new net N$4: R6.2
- new net N$9: R2.2, R3.2, S1-2.2, S1-3.2
- net +3V3: now also R5.2, R7.2; no longer R2.2
- net GND: now also R4.1, S1-4.2; no longer S1.P, S1.P1
- net N$1: no longer R1.2
- net N$5: now also S1-1.1, S1-2.1; no longer IC2_1W.1W
- net N$8: now also R1.2, R5.1, S1-1.2; no longer S1.S, S1.S1
Other:
- moved on the sheet: C1, IC1, IC2P, JP1, R1, R2

Commit message: Add files via upload
Parts:
- removed IC1: TINY25/45/85, atmel:TINY15LP
- added U$1: TINY25/45/85-20PU, avr-7:TINY25/45/85-20SU
- S1: value (none) -> Address
Connections:
- net +3V3: now also U$1.VCC; no longer IC1.VCC
- net GND: now also U$1.GND; no longer IC1.GND
- net N$1: now also U$1.(AREF)PB0; no longer IC1.(AREF)PB0
- net N$2: now also U$1.(ADC1)PB2; no longer IC1.(ADC1)PB2
- net N$3: now also U$1.(OCP)PB1; no longer IC1.(OCP)PB1
- net N$6: now also U$1.(ADC2)PB4; no longer IC1.(ADC3)PB4
- net N$7: now also U$1.(ADC0)PB5; no longer IC1.(ADC0)PB5
- net N$8: now also U$1.(ADC3)PB3; no longer IC1.(ADC2)PB3
Other:
- moved on the sheet: C1, R1, S1-1, S1-2, S1-3, S1-4
